File: dpt.kicad_sch (KiCad schematic)
At the start: 26 parts, among them J5 PT UPW 1, J6 PT UPW 2, J7 PT HFE 1, J8 PT HFE 2, U54 LTC4316CMS, U55 LTC4316CMS, U56 LTC4316CMS, U57 LTC4316CMS

Commit message: work
Parts:
- U56: renamed from U54; footprint Package_SO:MSOP-10_3x3mm_P0.5mm -> Package_DFN_QFN:DFN-10-1EP_3x3mm_P0.5mm_EP1.65x2.38mm
- U57: renamed from U56; footprint Package_SO:MSOP-10_3x3mm_P0.5mm -> Package_DFN_QFN:DFN-10-1EP_3x3mm_P0.5mm_EP1.65x2.38mm
- U58: renamed from U55; footprint Package_SO:MSOP-10_3x3mm_P0.5mm -> Package_DFN_QFN:DFN-10-1EP_3x3mm_P0.5mm_EP1.65x2.38mm
- U59: renamed from U57; footprint Package_SO:MSOP-10_3x3mm_P0.5mm -> Package_DFN_QFN:DFN-10-1EP_3x3mm_P0.5mm_EP1.65x2.38mm
- renumbered C108 to C104, C110 to C105, C109 to C106, C111 to C107, J7 to J6, J6 to J7, R243 to R237, R244 to R238, R237 to R239, R245 to R240, R238 to R241, R246 to R242, R241 to R243, R242 to R244, R247 to R245, R248 to R246, R239 to R247, R249 to R248, R240 to R249
