File: thrust-control-main.kicad_sch (KiCad schematic)
At the start: 18 parts, among them U20 MCP3208, U21 LTC2620IGN, U33 LM358, U34 LM358, U45 MAX6103, U46 LM358, U62 LM358

Commit message: work
Other:
- sheet Thrust Channel 1 ports: added none; removed OUT
- sheet Thrust Channel 2 ports: added none; removed OUT
- sheet Thrust Channel 3 ports: added none; removed OUT
- sheet Thrust Channel 4 ports: added none; removed OUT
- sheet Thrust Channel 5 ports: added none; removed OUT
- sheet Thrust Channel 6 ports: added none; removed OUT
- sheet Thrust Channel 7 ports: added none; removed OUT
- sheet Thrust Channel 8 ports: added none; removed OUT
- moved on the sheet: C81, C82, C92, C93, U33C, U34C, U46C, U62C

Commit message: 540 COMPONENTS I AM LOSING MY MINDDDDDD
Parts:
- renumbered C40 to C22, C38 to C23, C45 to C24, C41 to C25, C42 to C26, C39 to C27, C81 to C28, C82 to C29, C92 to C30, C93 to C31, R84 to R33, U20 to U10, U21 to U11, U45 to U12, U33 to U13, U34 to U14, U46 to U15, U62 to U16
Connections:
- net ADC_CS renamed POUT_CS
- net DAC_CS renamed PSET_CS
Other:
- moved on the sheet: C22, C23, C24, C25, C26, C27, C28, C29, C30, C31, R33, U10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

Commit message: schematic finished milestone
Parts:
- added C29: 10uF, symbol Device:C
- C28: renamed from C27; value 0.1uF -> 1uF
- renumbered C22 to C23, C23 to C24, C24 to C25, C25 to C26, C26 to C27, C28 to C30, C29 to C31, C30 to C32, C31 to C33, R33 to R42
Connections:
- net +3.3V: now also C29.1
- net GND: now also C29.2
Other:
- moved on the sheet: C23

Commit message: capacitor footprints
Parts:
- C23, C24, C25, C26, C27, C28, C30, C31, C32, C33: footprint (none) -> Capacitor_SMD:C_0603_1608Metric
- C29: footprint (none) -> Capacitor_SMD:C_0805_2012Metric
Changed lines of the file:
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@@
 			)
 		)
-		(property "Footprint" ""
+		(property "Footprint" "Capacitor_SMD:C_0603_1608Metric"
 			(at 180.0352 50.8 0)
 			(effects
@@
 			)
 		)
-		(property "Footprint" ""
+		(property "Footprint" "Capacitor_SMD:C_0603_1608Metric"
 			(at 84.7852 91.44 0)
 			(effects
@@
 			)
 		)
-		(property "Footprint" ""
+		(property "Footprint" "Capacitor_SMD:C_0603_1608Metric"
 			(at 51.7652 91.44 0)
 			(effects
@@
 			)
 		)
-		(property "Footprint" ""
+		(property "Footprint" "Capacitor_SMD:C_0603_1608Metric"
 			(at 77.1652 151.13 0)
 			(effects
@@
 			)
 		)
-		(property "Footprint" ""
+		(property "Footprint" "Capacitor_SMD:C_0603_1608Metric"
 			(at 82.2452 63.5 0)
 			(effects
@@
 			)
 		)
-		(property "Footprint" ""
+		(property "Footprint" "Capacitor_SMD:C_0603_1608Metric"
 			(at 180.0352 139.7 0)
 			(effects
@@
 			)
 		)
-		(property "Footprint" ""
+		(property "Footprint" "Capacitor_SMD:C_0603_1608Metric"
 			(at 180.0352 110.49 0)
 			(effects
@@
 			)
 		)
-		(property "Footprint" ""
+		(property "Footprint" "Capacitor_SMD:C_0603_1608Metric"
 			(at 53.0352 59.69 0)
 			(effects
@@
 			)
 		)
-		(property "Footprint" ""
+		(property "Footprint" "Capacitor_SMD:C_0603_1608Metric"
 			(at 180.0352 80.01 0)
 			(effects
@@
 			)
 		)
-		(property "Footprint" ""
+		(property "Footprint" "Capacitor_SMD:C_0805_2012Metric"
 			(at 96.2152 91.44 0)
 			(effects
@@
 			)
 		)
-		(property "Footprint" ""
+		(property "Footprint" "Capacitor_SMD:C_0603_1608Metric"
 			(at 40.3352 151.13 0)
 			(effects

Commit message: add more footprints
Parts:
- R42: footprint (none) -> Resistor_SMD:R_0603_1608Metric
- U11: footprint (none) -> Package_SO:SSOP-16_3.9x4.9mm_P0.635mm
- U13, U14, U15, U16: footprint (none) -> Package_SO:SOIC-8_3.9x4.9mm_P1.27mm
Changed lines of the file:
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@@
 			)
 		)
-		(property "Footprint" ""
+		(property "Footprint" "Package_SO:SOIC-8_3.9x4.9mm_P1.27mm"
 			(at 193.04 46.99 0)
 			(effects
@@
 			)
 		)
-		(property "Footprint" ""
+		(property "Footprint" "Package_SO:SOIC-8_3.9x4.9mm_P1.27mm"
 			(at 193.04 76.2 0)
 			(effects
@@
 			)
 		)
-		(property "Footprint" ""
+		(property "Footprint" "Package_SO:SOIC-8_3.9x4.9mm_P1.27mm"
 			(at 193.04 106.68 0)
 			(effects
@@
 			)
 		)
-		(property "Footprint" ""
+		(property "Footprint" "Resistor_SMD:R_0603_1608Metric"
 			(at 52.578 156.21 90)
 			(effects
@@
 			)
 		)
-		(property "Footprint" ""
+		(property "Footprint" "Package_SO:SSOP-16_3.9x4.9mm_P0.635mm"
 			(at 63.5 154.94 0)
 			(effects
@@
 			)
 		)
-		(property "Footprint" ""
+		(property "Footprint" "Package_SO:SOIC-8_3.9x4.9mm_P1.27mm"
 			(at 193.04 135.89 0)
 			(effects
