File: thrust-control-side.kicad_sch (KiCad schematic)
At the start: 11 parts, among them U22 MCP3204, U23 LM358, U60 LTC2622, U76 MAX6103

Commit message: work
Connections:
- net GND: now also U22.3 (CH2)
Other:
- sheet Thrust Channel 1 ports: added none; removed OUT
- sheet Thrust Channel 2 ports: added none; removed OUT
Changed lines of the file:
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@@
 	(paper "A4")
+	(junction
+		(at 163.83 62.23)
+		(diameter 0)
+		(color 0 0 0 0)
+	)
 	(junction
 		(at 90.17 19.05)
@@
 	(wire
 		(pts
-			(xy 54.61 95.25) (xy 64.77 95.25)
+			(xy 54.61 91.44) (xy 64.77 91.44)
 		)
 		(stroke
@@
 	(wire
 		(pts
-			(xy 104.14 99.06) (xy 93.98 99.06)
+			(xy 104.14 91.44) (xy 93.98 91.44)
 		)
 		(stroke
@@
 	(wire
 		(pts
+			(xy 163.83 59.69) (xy 163.83 62.23)
+		)
+		(stroke
+			(width 0)
+			(type default)
+		)
+	)
+	(wire
+		(pts
 			(xy 163.83 69.85) (xy 176.53 69.85)
 		)
@@
 	(wire
 		(pts
-			(xy 104.14 85.09) (xy 93.98 85.09)
+			(xy 104.14 81.28) (xy 93.98 81.28)
 		)
 		(stroke
@@
 	(wire
 		(pts
-			(xy 104.14 81.28) (xy 93.98 81.28)
-		)
-		(stroke
-			(width 0)
-			(type default)
-		)
-	)
-	(wire
-		(pts
 			(xy 194.31 54.61) (xy 204.47 54.61)
 		)
@@
 		(pts
 			(xy 179.07 35.56) (xy 179.07 46.99)
-		)
-		(stroke
-			(width 0)
-			(type default)
-		)
-	)
-	(wire
-		(pts
-			(xy 104.14 95.25) (xy 93.98 95.25)
 		)
 		(stroke
@@
 	)
 	(label "POUT_2"
-		(at 104.14 99.06 180)
+		(at 104.14 91.44 180)
 		(fields_autoplaced yes)
 		(effects
@@
 		)
 	)
-	(label "OUT_2"
-		(at 104.14 95.25 180)
+	(label "POUT_1"
+		(at 153.67 54.61 0)
 		(fields_autoplaced yes)
 		(effects
@@
 				(size 1.27 1.27)
 			)
-			(justify right bottom)
-		)
-	)
-	(label "POUT_1"
-		(at 153.67 54.61 0)
+			(justify left bottom)
+		)
+	)
+	(label "PSET_1"
+		(at 54.61 81.28 0)
 		(fields_autoplaced yes)
 		(effects
@@
 		)
 	)
-	(label "PSET_1"
-		(at 54.61 81.28 0)
+	(label "3V_REF"
+		(at 156.21 35.56 0)
 		(fields_autoplaced yes)
 		(effects
@@
 		)
 	)
-	(label "3V_REF"
-		(at 156.21 35.56 0)
+	(label "SPI_MISO"
+		(at 204.47 57.15 180)
 		(fields_autoplaced yes)
 		(effects
@@
 				(size 1.27 1.27)
 			)
-			(justify left bottom)
-		)
-	)
-	(label "SPI_MISO"
-		(at 204.47 57.15 180)
+			(justify right bottom)
+		)
+	)
+	(label "ADC_CS"
+		(at 204.47 62.23 180)
 		(fields_autoplaced yes)
 		(effects
@@
 		)
 	)
-	(label "ADC_CS"
-		(at 204.47 62.23 180)
+	(label "3V_REF"
+		(at 115.57 19.05 180)
 		(fields_autoplaced yes)
 		(effects
@@
 		)
 	)
-	(label "3V_REF"
-		(at 115.57 19.05 180)
+	(label "SPI_MOSI"
+		(at 204.47 59.69 180)
 		(fields_autoplaced yes)
 		(effects
@@
 		)
 	)
-	(label "SPI_MOSI"
-		(at 204.47 59.69 180)
+	(label "PSET_2"
+		(at 114.3 44.45 180)
 		(fields_autoplaced yes)
 		(effects
@@
 		)
 	)
-	(label "PSET_2"
-		(at 114.3 44.45 180)
+	(label "POUT_2"
+		(at 153.67 57.15 0)
 		(fields_autoplaced yes)
 		(effects
@@
 				(size 1.27 1.27)
 			)
-			(justify right bottom)
-		)
-	)
-	(label "POUT_2"
-		(at 153.67 57.15 0)
+			(justify left bottom)
+		)
+	)
+	(label "DAC_CS"
+		(at 71.12 46.99 0)
 		(fields_autoplaced yes)
 		(effects
@@
 		)
 	)
-	(label "DAC_CS"
-		(at 71.12 46.99 0)
+	(label "3V_REF"
+		(at 62.23 36.83 180)
 		(fields_autoplaced yes)
 		(effects
@@
 				(size 1.27 1.27)
 			)
-			(justify left bottom)
-		)
-	)
-	(label "3V_REF"
-		(at 62.23 36.83 180)
+			(justify right bottom)
+		)
+	)
+	(label "PSET_2"
+		(at 54.61 91.44 0)
 		(fields_autoplaced yes)
 		(effects
@@
 				(size 1.27 1.27)
 			)
-			(justify right bottom)
-		)
-	)
-	(label "PSET_2"
-		(at 54.61 95.25 0)
+			(justify left bottom)
+		)
+	)
+	(label "SPI_SCK"
+		(at 204.47 54.61 180)
 		(fields_autoplaced yes)
 		(effects
@@
 				(size 1.27 1.27)
 			)
-			(justify left bottom)
-		)
-	)
-	(label "SPI_SCK"
-		(at 204.47 54.61 180)
+			(justify right bottom)
+		)
+	)
+	(label "SPI_MOSI"
+		(at 71.12 41.91 0)
 		(fields_autoplaced yes)
 		(effects
@@
 				(size 1.27 1.27)
 			)
-			(justify right bottom)
-		)
-	)
-	(label "OUT_1"
+			(justify left bottom)
+		)
+	)
+	(label "POUT_1"
 		(at 104.14 81.28 180)
-		(fields_autoplaced yes)
-		(effects
-			(font
-				(size 1.27 1.27)
-			)
-			(justify right bottom)
-		)
-	)
-	(label "SPI_MOSI"
-		(at 71.12 41.91 0)
-		(fields_autoplaced yes)
-		(effects
-			(font
-				(size 1.27 1.27)
-			)
-			(justify left bottom)
-		)
-	)
-	(label "POUT_1"
-		(at 104.14 85.09 180)
 		(fields_autoplaced yes)
 		(effects
@@
 	(sheet
 		(at 64.77 78.74)
-		(size 29.21 8.89)
+		(size 29.21 5.08)
 		(fields_autoplaced yes)
 		(stroke
@@
 		)
 		(property "Sheetfile" "thrust-channel.kicad_sch"
-			(at 64.77 88.2146 0)
+			(at 64.77 84.4046 0)
 			(effects
 				(font
@@
 		)
 		(pin "TELEM_POUT" output
-			(at 93.98 85.09 0)
-			(effects
-				(font
-					(size 1.27 1.27)
-				)
-				(justify right)
-			)
-		)
-		(pin "OUT" output
 			(at 93.98 81.28 0)
 			(effects
@@
 	)
 	(sheet
-		(at 64.77 92.71)
-		(size 29.21 8.89)
+		(at 64.77 88.9)
+		(size 29.21 5.08)
 		(fields_autoplaced yes)
 		(stroke
@@
 		)
 		(property "Sheetname" "Thrust Channel 2"
-			(at 64.77 91.9984 0)
+			(at 64.77 88.1884 0)
 			(effects
 				(font
@@
 		)
 		(property "Sheetfile" "thrust-channel.kicad_sch"
-			(at 64.77 102.1846 0)
+			(at 64.77 94.5646 0)
 			(effects
 				(font
@@
 		)
 		(pin "PSET" input
-			(at 64.77 95.25 180)
+			(at 64.77 91.44 180)
 			(effects
 				(font
@@
 		)
 		(pin "TELEM_POUT" output
-			(at 93.98 99.06 0)
-			(effects
-				(font
-					(size 1.27 1.27)
-				)
-				(justify right)
-			)
-		)
-		(pin "OUT" output
-			(at 93.98 95.25 0)
-			(effects
-				(font
+			(at 93.98 91.44 0)
+			(effects
+				(font

Commit message: lots and lots and lots of work
Connections:
- net SPI_SCK renamed SPI_CLK
Changed lines of the file:
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@@
 		)
 	)
-	(label "SPI_SCK"
+	(label "SPI_CLK"
 		(at 71.12 39.37 0)
 		(fields_autoplaced yes)
@@
 		)
 	)
-	(label "SPI_SCK"
+	(label "SPI_CLK"
 		(at 204.47 54.61 180)
 		(fields_autoplaced yes)
@@
 			(project "femta-control"
 				(path "/838bf11c-36b7-41d7-9462-fe98a188d617/c8752098-45e2-4d20-a718-e7a412b889c5"
-					(page "9")
-				)
-				(path "/838bf11c-36b7-41d7-9462-fe98a188d617/25504b25-63a2-43d8-9fee-c553eccedd0e"
-					(page "13")
+					(page "20")
+				)
+				(path "/838bf11c-36b7-41d7-9462-fe98a188d617/25504b25-63a2-43d8-9fee-c553eccedd0e"
+					(page "17")
 				)
 			)
@@
 			(project "femta-control"
 				(path "/838bf11c-36b7-41d7-9462-fe98a188d617/c8752098-45e2-4d20-a718-e7a412b889c5"
-					(page "10")
-				)
-				(path "/838bf11c-36b7-41d7-9462-fe98a188d617/25504b25-63a2-43d8-9fee-c553eccedd0e"
-					(page "15")
-				)
-			)
+					(page "21")
+				)
+				(path "/838bf11c-36b7-41d7-9462-fe98a188d617/25504b25-63a2-43d8-9fee-c553eccedd0e"
+					(page "18")
+				)
+			)

Commit message: 540 COMPONENTS I AM LOSING MY MINDDDDDD
Parts:
- renumbered C54 to C49, C55 to C50, C46 to C51, C50 to C52, C51 to C53, C58 to C54, C59 to C55, U23 to U38, U76 to U42, U60 to U43, U22 to U44
Connections:
- net ADC_CS renamed POUT_CS
- net DAC_CS renamed PSET_CS
Other:
- moved on the sheet: C51, C52, C53, U38C, U43

Commit message: schematic finished milestone
Parts:
- added C49: 10uF, symbol Device:C
- C58: renamed from C55; value 0.1uF -> 1uF
- renumbered C49 to C52, C50 to C53, C51 to C54, C52 to C55, C53 to C56, C54 to C57, U42 to U41, U38 to U42
Connections:
- net +3.3V: now also C49.1
- net GND: now also C49.2
Other:
- moved on the sheet: C55

Commit message: capacitor footprints
Parts:
- C49: footprint (none) -> Capacitor_SMD:C_0805_2012Metric
- C52, C53, C54, C55, C56, C57, C58: footprint (none) -> Capacitor_SMD:C_0603_1608Metric
Changed lines of the file:
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@@
 			)
 		)
-		(property "Footprint" ""
+		(property "Footprint" "Capacitor_SMD:C_0603_1608Metric"
 			(at 167.3352 43.18 0)
 			(effects
@@
 			)
 		)
-		(property "Footprint" ""
+		(property "Footprint" "Capacitor_SMD:C_0603_1608Metric"
 			(at 121.6152 36.83 0)
 			(effects
@@
 			)
 		)
-		(property "Footprint" ""
+		(property "Footprint" "Capacitor_SMD:C_0603_1608Metric"
 			(at 195.2752 43.18 0)
 			(effects
@@
 			)
 		)
-		(property "Footprint" ""
+		(property "Footprint" "Capacitor_SMD:C_0603_1608Metric"
 			(at 84.7852 36.83 0)
 			(effects
@@
 			)
 		)
-		(property "Footprint" ""
+		(property "Footprint" "Capacitor_SMD:C_0603_1608Metric"
 			(at 58.1152 88.9 0)
 			(effects
@@
 			)
 		)
-		(property "Footprint" ""
+		(property "Footprint" "Capacitor_SMD:C_0603_1608Metric"
 			(at 54.3052 44.45 0)
 			(effects
@@
 			)
 		)
-		(property "Footprint" ""
+		(property "Footprint" "Capacitor_SMD:C_0603_1608Metric"
 			(at 25.0952 40.64 0)
 			(effects
@@
 			)
 		)
-		(property "Footprint" ""
+		(property "Footprint" "Capacitor_SMD:C_0805_2012Metric"
 			(at 206.7052 43.18 0)
 			(effects

Commit message: add more footprints
Parts:
- U42: footprint (none) -> Package_SO:SOIC-8_3.9x4.9mm_P1.27mm
Changed lines of the file:
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@@
 			)
 		)
-		(property "Footprint" ""
+		(property "Footprint" "Package_SO:SOIC-8_3.9x4.9mm_P1.27mm"
 			(at 71.12 85.09 0)
 			(effects
