File: LCL_HV.kicad_sch (KiCad schematic)
At the start: 7 parts, among them Q19 DMP4015SSSQ-13, Q20 MMBT3904, U37 INA202DGK-Q1

Commit message: work
Parts:
- renumbered C94 to C79, Q20 to Q16, Q19 to Q17, R130 to R133, R131 to R134, U37 to U31
Changed lines of the file:
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@@
 		(on_board yes)
 		(dnp no)
-		(property "Reference" "#PWR0194"
+		(property "Reference" "#PWR0141"
 			(at 128.27 120.65 0)
 			(effects
@@
 			(project "femta-control"
 				(path "/838bf11c-36b7-41d7-9462-fe98a188d617/85fed540-db98-47e1-a986-73b49dbf8bdb"
-					(reference "#PWR0194")
+					(reference "#PWR0141")
 					(unit 1)
 				)
@@
 		(on_board yes)
 		(dnp no)
-		(property "Reference" "C94"
+		(property "Reference" "C79"
 			(at 130.81 109.22 0)
 			(effects
@@
 			(project "femta-control"
 				(path "/838bf11c-36b7-41d7-9462-fe98a188d617/85fed540-db98-47e1-a986-73b49dbf8bdb"
-					(reference "C94")
+					(reference "C79")
 					(unit 1)
 				)
@@
 		(on_board yes)
 		(dnp no)
-		(property "Reference" "R131"
+		(property "Reference" "R134"
 			(at 185.42 90.17 0)
 			(effects
@@
 			(project "femta-control"
 				(path "/838bf11c-36b7-41d7-9462-fe98a188d617/85fed540-db98-47e1-a986-73b49dbf8bdb"
-					(reference "R131")
+					(reference "R134")
 					(unit 1)
 				)
@@
 		(dnp no)
 		(fields_autoplaced yes)
-		(property "Reference" "Q19"
+		(property "Reference" "Q17"
 			(at 191.77 73.66 90)
 			(effects
@@
 			(project "femta-control"
 				(path "/838bf11c-36b7-41d7-9462-fe98a188d617/85fed540-db98-47e1-a986-73b49dbf8bdb"
-					(reference "Q19")
+					(reference "Q17")
 					(unit 1)
 				)
@@
 		(dnp no)
 		(fields_autoplaced yes)
-		(property "Reference" "Q20"
+		(property "Reference" "Q16"
 			(at 194.31 105.4099 0)
 			(effects
@@
 			(project "femta-control"
 				(path "/838bf11c-36b7-41d7-9462-fe98a188d617/85fed540-db98-47e1-a986-73b49dbf8bdb"
-					(reference "Q20")
+					(reference "Q16")
 					(unit 1)
 				)
@@
 		(on_board yes)
 		(dnp no)
-		(property "Reference" "#PWR0195"
+		(property "Reference" "#PWR0142"
 			(at 151.13 152.4 0)
 			(effects
@@
 			(project "femta-control"
 				(path "/838bf11c-36b7-41d7-9462-fe98a188d617/85fed540-db98-47e1-a986-73b49dbf8bdb"
-					(reference "#PWR0195")
+					(reference "#PWR0142")
 					(unit 1)
 				)
@@
 		(dnp no)
 		(fields_autoplaced yes)
-		(property "Reference" "U37"
+		(property "Reference" "U31"
 			(at 153.3241 110.49 0)
 			(effects
@@
 			(project "femta-control"
 				(path "/838bf11c-36b7-41d7-9462-fe98a188d617/85fed540-db98-47e1-a986-73b49dbf8bdb"
-					(reference "U37")
+					(reference "U31")
 					(unit 1)
 				)
@@
 		(on_board yes)
 		(dnp no)
-		(property "Reference" "R130"
+		(property "Reference" "R133"
 			(at 177.8 77.724 90)
 			(effects
@@
 			(project "femta-control"
 				(path "/838bf11c-36b7-41d7-9462-fe98a188d617/85fed540-db98-47e1-a986-73b49dbf8bdb"
-					(reference "R130")
-					(unit 1)
-				)
+					(reference "R133")
+					(unit 1)
+				)

Commit message: 540 COMPONENTS I AM LOSING MY MINDDDDDD
Parts:
- renumbered C79 to C20, Q16 to Q3, Q17 to Q4, R132 to R28, R133 to R29, R134 to R30, U31 to U8
Changed lines of the file:
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@@
 		(on_board yes)
 		(dnp no)
-		(property "Reference" "#PWR0141"
+		(property "Reference" "#PWR046"
 			(at 128.27 120.65 0)
 			(effects
@@
 			(project "femta-control"
 				(path "/838bf11c-36b7-41d7-9462-fe98a188d617/85fed540-db98-47e1-a986-73b49dbf8bdb"
-					(reference "#PWR0141")
+					(reference "#PWR046")
 					(unit 1)
 				)
@@
 		(on_board yes)
 		(dnp no)
-		(property "Reference" "R132"
+		(property "Reference" "R28"
 			(at 167.64 104.394 90)
 			(effects
@@
 			(project "femta-control"
 				(path "/838bf11c-36b7-41d7-9462-fe98a188d617/85fed540-db98-47e1-a986-73b49dbf8bdb"
-					(reference "R132")
+					(reference "R28")
 					(unit 1)
 				)
@@
 		(on_board yes)
 		(dnp no)
-		(property "Reference" "C79"
+		(property "Reference" "C20"
 			(at 130.81 109.22 0)
 			(effects
@@
 			(project "femta-control"
 				(path "/838bf11c-36b7-41d7-9462-fe98a188d617/85fed540-db98-47e1-a986-73b49dbf8bdb"
-					(reference "C79")
+					(reference "C20")
 					(unit 1)
 				)
@@
 		(on_board yes)
 		(dnp no)
-		(property "Reference" "R134"
+		(property "Reference" "R30"
 			(at 185.42 90.17 0)
 			(effects
@@
 			(project "femta-control"
 				(path "/838bf11c-36b7-41d7-9462-fe98a188d617/85fed540-db98-47e1-a986-73b49dbf8bdb"
-					(reference "R134")
+					(reference "R30")
 					(unit 1)
 				)
@@
 		(dnp no)
 		(fields_autoplaced yes)
-		(property "Reference" "Q17"
+		(property "Reference" "Q4"
 			(at 191.77 73.66 90)
 			(effects
@@
 			(project "femta-control"
 				(path "/838bf11c-36b7-41d7-9462-fe98a188d617/85fed540-db98-47e1-a986-73b49dbf8bdb"
-					(reference "Q17")
+					(reference "Q4")
 					(unit 1)
 				)
@@
 		(dnp no)
 		(fields_autoplaced yes)
-		(property "Reference" "Q16"
+		(property "Reference" "Q3"
 			(at 194.31 105.4099 0)
 			(effects
@@
 			(project "femta-control"
 				(path "/838bf11c-36b7-41d7-9462-fe98a188d617/85fed540-db98-47e1-a986-73b49dbf8bdb"
-					(reference "Q16")
+					(reference "Q3")
 					(unit 1)
 				)
@@
 		(on_board yes)
 		(dnp no)
-		(property "Reference" "#PWR0142"
+		(property "Reference" "#PWR047"
 			(at 151.13 152.4 0)
 			(effects
@@
 			(project "femta-control"
 				(path "/838bf11c-36b7-41d7-9462-fe98a188d617/85fed540-db98-47e1-a986-73b49dbf8bdb"
-					(reference "#PWR0142")
+					(reference "#PWR047")
 					(unit 1)
 				)
@@
 		(dnp no)
 		(fields_autoplaced yes)
-		(property "Reference" "U31"
+		(property "Reference" "U8"
 			(at 153.3241 110.49 0)
 			(effects
@@
 			(project "femta-control"
 				(path "/838bf11c-36b7-41d7-9462-fe98a188d617/85fed540-db98-47e1-a986-73b49dbf8bdb"
-					(reference "U31")
+					(reference "U8")
 					(unit 1)
 				)
@@
 		(on_board yes)
 		(dnp no)
-		(property "Reference" "R133"
+		(property "Reference" "R29"
 			(at 177.8 77.724 90)
 			(effects
@@
 			(project "femta-control"
 				(path "/838bf11c-36b7-41d7-9462-fe98a188d617/85fed540-db98-47e1-a986-73b49dbf8bdb"
-					(reference "R133")
-					(unit 1)
-				)
+					(reference "R29")
+					(unit 1)
+				)

Commit message: schematic finished milestone
Parts:
- renumbered C20 to C21, R28 to R37, R29 to R38, R30 to R39
Changed lines of the file:
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@@
 		(on_board yes)
 		(dnp no)
-		(property "Reference" "#PWR046"
+		(property "Reference" "#PWR047"
 			(at 128.27 120.65 0)
 			(effects
@@
 			(project "femta-control"
 				(path "/838bf11c-36b7-41d7-9462-fe98a188d617/85fed540-db98-47e1-a986-73b49dbf8bdb"
-					(reference "#PWR046")
+					(reference "#PWR047")
 					(unit 1)
 				)
@@
 		(on_board yes)
 		(dnp no)
-		(property "Reference" "R28"
+		(property "Reference" "R37"
 			(at 167.64 104.394 90)
 			(effects
@@
 			(project "femta-control"
 				(path "/838bf11c-36b7-41d7-9462-fe98a188d617/85fed540-db98-47e1-a986-73b49dbf8bdb"
-					(reference "R28")
+					(reference "R37")
 					(unit 1)
 				)
@@
 		(on_board yes)
 		(dnp no)
-		(property "Reference" "C20"
+		(property "Reference" "C21"
 			(at 130.81 109.22 0)
 			(effects
@@
 			(project "femta-control"
 				(path "/838bf11c-36b7-41d7-9462-fe98a188d617/85fed540-db98-47e1-a986-73b49dbf8bdb"
-					(reference "C20")
+					(reference "C21")
 					(unit 1)
 				)
@@
 		(on_board yes)
 		(dnp no)
-		(property "Reference" "R30"
+		(property "Reference" "R39"
 			(at 185.42 90.17 0)
 			(effects
@@
 			(project "femta-control"
 				(path "/838bf11c-36b7-41d7-9462-fe98a188d617/85fed540-db98-47e1-a986-73b49dbf8bdb"
-					(reference "R30")
+					(reference "R39")
 					(unit 1)
 				)
@@
 		(on_board yes)
 		(dnp no)
-		(property "Reference" "#PWR047"
+		(property "Reference" "#PWR048"
 			(at 151.13 152.4 0)
 			(effects
@@
 			(project "femta-control"
 				(path "/838bf11c-36b7-41d7-9462-fe98a188d617/85fed540-db98-47e1-a986-73b49dbf8bdb"
-					(reference "#PWR047")
+					(reference "#PWR048")
 					(unit 1)
 				)
@@
 		(on_board yes)
 		(dnp no)
-		(property "Reference" "R29"
+		(property "Reference" "R38"
 			(at 177.8 77.724 90)
 			(effects
@@
 			(project "femta-control"
 				(path "/838bf11c-36b7-41d7-9462-fe98a188d617/85fed540-db98-47e1-a986-73b49dbf8bdb"
-					(reference "R29")
-					(unit 1)
-				)
+					(reference "R38")
+					(unit 1)
+				)

Commit message: capacitor footprints
Parts:
- C21: footprint (none) -> Capacitor_SMD:C_0603_1608Metric
Changed lines of the file:
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@@
 			)
 		)
-		(property "Footprint" ""
+		(property "Footprint" "Capacitor_SMD:C_0603_1608Metric"
 			(at 129.2352 114.3 0)
 			(effects

Commit message: add more footprints
Parts:
- R37, R39: footprint (none) -> Resistor_SMD:R_0603_1608Metric
Changed lines of the file:
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@@
 			)
 		)
-		(property "Footprint" ""
+		(property "Footprint" "Resistor_SMD:R_0603_1608Metric"
 			(at 167.64 108.458 90)
 			(effects
@@
 			)
 		)
-		(property "Footprint" ""
+		(property "Footprint" "Resistor_SMD:R_0603_1608Metric"
 			(at 182.372 90.17 90)
 			(effects

Commit message: footprint selection
Parts:
- R38: footprint (none) -> Resistor_SMD:R_0805_2012Metric
Changed lines of the file:
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@@
 			)
 		)
-		(property "Footprint" ""
+		(property "Footprint" "Resistor_SMD:R_0805_2012Metric"
 			(at 177.8 81.788 90)
 			(effects
