File: LCL_LV.kicad_sch (KiCad schematic)
At the start: 5 parts, among them Q18 DMP4015SSSQ-13, U35 INA202DGK-Q1

Commit message: work
Parts:
- renumbered C93 to C78, Q18 to Q15, R123 to R129, R128 to R130, U35 to U29
Changed lines of the file:
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@@
 		(dnp no)
 		(fields_autoplaced yes)
-		(property "Reference" "U35"
+		(property "Reference" "U29"
 			(at 125.3841 83.82 0)
 			(effects
@@
 			(project "femta-control"
 				(path "/838bf11c-36b7-41d7-9462-fe98a188d617/2005ce18-3dfb-489b-ad6c-5d04a90f0ec8"
-					(reference "U35")
-					(unit 1)
-				)
-				(path "/838bf11c-36b7-41d7-9462-fe98a188d617/d7ed326e-dbc5-4110-8331-7e3bdacabdbd"
-					(reference "U36")
-					(unit 1)
-				)
-				(path "/838bf11c-36b7-41d7-9462-fe98a188d617/9caee5f1-c259-48c3-ab00-5902eb9cdfc4"
-					(reference "U38")
+					(reference "U29")
+					(unit 1)
+				)
+				(path "/838bf11c-36b7-41d7-9462-fe98a188d617/d7ed326e-dbc5-4110-8331-7e3bdacabdbd"
+					(reference "U30")
+					(unit 1)
+				)
+				(path "/838bf11c-36b7-41d7-9462-fe98a188d617/9caee5f1-c259-48c3-ab00-5902eb9cdfc4"
+					(reference "U32")
 					(unit 1)
 				)
@@
 		(on_board yes)
 		(dnp no)
-		(property "Reference" "C93"
+		(property "Reference" "C78"
 			(at 110.49 77.47 0)
 			(effects
@@
 			(project "femta-control"
 				(path "/838bf11c-36b7-41d7-9462-fe98a188d617/d7ed326e-dbc5-4110-8331-7e3bdacabdbd"
-					(reference "C93")
-					(unit 1)
-				)
-				(path "/838bf11c-36b7-41d7-9462-fe98a188d617/2005ce18-3dfb-489b-ad6c-5d04a90f0ec8"
-					(reference "C92")
-					(unit 1)
-				)
-				(path "/838bf11c-36b7-41d7-9462-fe98a188d617/9caee5f1-c259-48c3-ab00-5902eb9cdfc4"
-					(reference "C95")
+					(reference "C78")
+					(unit 1)
+				)
+				(path "/838bf11c-36b7-41d7-9462-fe98a188d617/2005ce18-3dfb-489b-ad6c-5d04a90f0ec8"
+					(reference "C77")
+					(unit 1)
+				)
+				(path "/838bf11c-36b7-41d7-9462-fe98a188d617/9caee5f1-c259-48c3-ab00-5902eb9cdfc4"
+					(reference "C80")
 					(unit 1)
 				)
@@
 		(dnp no)
 		(fields_autoplaced yes)
-		(property "Reference" "Q18"
+		(property "Reference" "Q15"
 			(at 163.83 68.58 90)
 			(effects
@@
 			(project "femta-control"
 				(path "/838bf11c-36b7-41d7-9462-fe98a188d617/d7ed326e-dbc5-4110-8331-7e3bdacabdbd"
+					(reference "Q15")
+					(unit 1)
+				)
+				(path "/838bf11c-36b7-41d7-9462-fe98a188d617/2005ce18-3dfb-489b-ad6c-5d04a90f0ec8"
+					(reference "Q14")
+					(unit 1)
+				)
+				(path "/838bf11c-36b7-41d7-9462-fe98a188d617/9caee5f1-c259-48c3-ab00-5902eb9cdfc4"
 					(reference "Q18")
-					(unit 1)
-				)
-				(path "/838bf11c-36b7-41d7-9462-fe98a188d617/2005ce18-3dfb-489b-ad6c-5d04a90f0ec8"
-					(reference "Q17")
-					(unit 1)
-				)
-				(path "/838bf11c-36b7-41d7-9462-fe98a188d617/9caee5f1-c259-48c3-ab00-5902eb9cdfc4"
-					(reference "Q21")
 					(unit 1)
 				)
@@
 		(on_board yes)
 		(dnp no)
-		(property "Reference" "R123"
+		(property "Reference" "R129"
 			(at 157.48 85.09 0)
 			(effects
@@
 			(project "femta-control"
 				(path "/838bf11c-36b7-41d7-9462-fe98a188d617/2005ce18-3dfb-489b-ad6c-5d04a90f0ec8"
-					(reference "R123")
-					(unit 1)
-				)
-				(path "/838bf11c-36b7-41d7-9462-fe98a188d617/d7ed326e-dbc5-4110-8331-7e3bdacabdbd"
 					(reference "R129")
 					(unit 1)
 				)
-				(path "/838bf11c-36b7-41d7-9462-fe98a188d617/9caee5f1-c259-48c3-ab00-5902eb9cdfc4"
-					(reference "R138")
+				(path "/838bf11c-36b7-41d7-9462-fe98a188d617/d7ed326e-dbc5-4110-8331-7e3bdacabdbd"
+					(reference "R131")
+					(unit 1)
+				)
+				(path "/838bf11c-36b7-41d7-9462-fe98a188d617/9caee5f1-c259-48c3-ab00-5902eb9cdfc4"
+					(reference "R136")
 					(unit 1)
 				)
@@
 		(on_board yes)
 		(dnp no)
-		(property "Reference" "R128"
+		(property "Reference" "R130"
 			(at 149.86 72.644 90)
 			(effects
@@
 			(project "femta-control"
 				(path "/838bf11c-36b7-41d7-9462-fe98a188d617/d7ed326e-dbc5-4110-8331-7e3bdacabdbd"
+					(reference "R130")
+					(unit 1)
+				)
+				(path "/838bf11c-36b7-41d7-9462-fe98a188d617/2005ce18-3dfb-489b-ad6c-5d04a90f0ec8"
 					(reference "R128")
 					(unit 1)
 				)
-				(path "/838bf11c-36b7-41d7-9462-fe98a188d617/2005ce18-3dfb-489b-ad6c-5d04a90f0ec8"
-					(reference "R121")
-					(unit 1)
-				)
-				(path "/838bf11c-36b7-41d7-9462-fe98a188d617/9caee5f1-c259-48c3-ab00-5902eb9cdfc4"
-					(reference "R137")
+				(path "/838bf11c-36b7-41d7-9462-fe98a188d617/9caee5f1-c259-48c3-ab00-5902eb9cdfc4"
+					(reference "R135")
 					(unit 1)
 				)
@@
 		(on_board yes)
 		(dnp no)
-		(property "Reference" "#PWR0192"
+		(property "Reference" "#PWR0139"
 			(at 107.95 88.9 0)
 			(effects
@@
 			(project "femta-control"
 				(path "/838bf11c-36b7-41d7-9462-fe98a188d617/d7ed326e-dbc5-4110-8331-7e3bdacabdbd"
-					(reference "#PWR0192")
-					(unit 1)
-				)
-				(path "/838bf11c-36b7-41d7-9462-fe98a188d617/2005ce18-3dfb-489b-ad6c-5d04a90f0ec8"
-					(reference "#PWR0188")
-					(unit 1)
-				)
-				(path "/838bf11c-36b7-41d7-9462-fe98a188d617/9caee5f1-c259-48c3-ab00-5902eb9cdfc4"
-					(reference "#PWR0200")
+					(reference "#PWR0139")
+					(unit 1)
+				)
+				(path "/838bf11c-36b7-41d7-9462-fe98a188d617/2005ce18-3dfb-489b-ad6c-5d04a90f0ec8"
+					(reference "#PWR0137")
+					(unit 1)
+				)
+				(path "/838bf11c-36b7-41d7-9462-fe98a188d617/9caee5f1-c259-48c3-ab00-5902eb9cdfc4"
+					(reference "#PWR0143")
 					(unit 1)
 				)
@@
 		(on_board yes)
 		(dnp no)
-		(property "Reference" "#PWR0189"
+		(property "Reference" "#PWR0138"
 			(at 123.19 125.73 0)
 			(effects
@@
 			(project "femta-control"
 				(path "/838bf11c-36b7-41d7-9462-fe98a188d617/2005ce18-3dfb-489b-ad6c-5d04a90f0ec8"
-					(reference "#PWR0189")
-					(unit 1)
-				)
-				(path "/838bf11c-36b7-41d7-9462-fe98a188d617/d7ed326e-dbc5-4110-8331-7e3bdacabdbd"
-					(reference "#PWR0193")
-					(unit 1)
-				)
-				(path "/838bf11c-36b7-41d7-9462-fe98a188d617/9caee5f1-c259-48c3-ab00-5902eb9cdfc4"
-					(reference "#PWR0201")
-					(unit 1)
-				)
+					(reference "#PWR0138")
+					(unit 1)
+				)
+				(path "/838bf11c-36b7-41d7-9462-fe98a188d617/d7ed326e-dbc5-4110-8331-7e3bdacabdbd"
+					(reference "#PWR0140")
+					(unit 1)
+				)
+				(path "/838bf11c-36b7-41d7-9462-fe98a188d617/9caee5f1-c259-48c3-ab00-5902eb9cdfc4"
+					(reference "#PWR0144")
+					(unit 1)
+				)

Commit message: 540 COMPONENTS I AM LOSING MY MINDDDDDD
Parts:
- renumbered C78 to C19, Q15 to Q2, R129 to R25, R130 to R26, U29 to U6
Changed lines of the file:
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@@
 		(dnp no)
 		(fields_autoplaced yes)
-		(property "Reference" "U29"
+		(property "Reference" "U6"
 			(at 125.3841 83.82 0)
 			(effects
@@
 			(project "femta-control"
 				(path "/838bf11c-36b7-41d7-9462-fe98a188d617/2005ce18-3dfb-489b-ad6c-5d04a90f0ec8"
-					(reference "U29")
-					(unit 1)
-				)
-				(path "/838bf11c-36b7-41d7-9462-fe98a188d617/d7ed326e-dbc5-4110-8331-7e3bdacabdbd"
-					(reference "U30")
-					(unit 1)
-				)
-				(path "/838bf11c-36b7-41d7-9462-fe98a188d617/9caee5f1-c259-48c3-ab00-5902eb9cdfc4"
-					(reference "U32")
+					(reference "U6")
+					(unit 1)
+				)
+				(path "/838bf11c-36b7-41d7-9462-fe98a188d617/d7ed326e-dbc5-4110-8331-7e3bdacabdbd"
+					(reference "U7")
+					(unit 1)
+				)
+				(path "/838bf11c-36b7-41d7-9462-fe98a188d617/9caee5f1-c259-48c3-ab00-5902eb9cdfc4"
+					(reference "U9")
 					(unit 1)
 				)
@@
 		(on_board yes)
 		(dnp no)
-		(property "Reference" "C78"
+		(property "Reference" "C19"
 			(at 110.49 77.47 0)
 			(effects
@@
 			(project "femta-control"
 				(path "/838bf11c-36b7-41d7-9462-fe98a188d617/d7ed326e-dbc5-4110-8331-7e3bdacabdbd"
-					(reference "C78")
-					(unit 1)
-				)
-				(path "/838bf11c-36b7-41d7-9462-fe98a188d617/2005ce18-3dfb-489b-ad6c-5d04a90f0ec8"
-					(reference "C77")
-					(unit 1)
-				)
-				(path "/838bf11c-36b7-41d7-9462-fe98a188d617/9caee5f1-c259-48c3-ab00-5902eb9cdfc4"
-					(reference "C80")
+					(reference "C19")
+					(unit 1)
+				)
+				(path "/838bf11c-36b7-41d7-9462-fe98a188d617/2005ce18-3dfb-489b-ad6c-5d04a90f0ec8"
+					(reference "C18")
+					(unit 1)
+				)
+				(path "/838bf11c-36b7-41d7-9462-fe98a188d617/9caee5f1-c259-48c3-ab00-5902eb9cdfc4"
+					(reference "C21")
 					(unit 1)
 				)
@@
 		(dnp no)
 		(fields_autoplaced yes)
-		(property "Reference" "Q15"
+		(property "Reference" "Q2"
 			(at 163.83 68.58 90)
 			(effects
@@
 			(project "femta-control"
 				(path "/838bf11c-36b7-41d7-9462-fe98a188d617/d7ed326e-dbc5-4110-8331-7e3bdacabdbd"
-					(reference "Q15")
-					(unit 1)
-				)
-				(path "/838bf11c-36b7-41d7-9462-fe98a188d617/2005ce18-3dfb-489b-ad6c-5d04a90f0ec8"
-					(reference "Q14")
-					(unit 1)
-				)
-				(path "/838bf11c-36b7-41d7-9462-fe98a188d617/9caee5f1-c259-48c3-ab00-5902eb9cdfc4"
-					(reference "Q18")
+					(reference "Q2")
+					(unit 1)
+				)
+				(path "/838bf11c-36b7-41d7-9462-fe98a188d617/2005ce18-3dfb-489b-ad6c-5d04a90f0ec8"
+					(reference "Q1")
+					(unit 1)
+				)
+				(path "/838bf11c-36b7-41d7-9462-fe98a188d617/9caee5f1-c259-48c3-ab00-5902eb9cdfc4"
+					(reference "Q5")
 					(unit 1)
 				)
@@
 		(on_board yes)
 		(dnp no)
-		(property "Reference" "R129"
+		(property "Reference" "R25"
 			(at 157.48 85.09 0)
 			(effects
@@
 			(project "femta-control"
 				(path "/838bf11c-36b7-41d7-9462-fe98a188d617/2005ce18-3dfb-489b-ad6c-5d04a90f0ec8"
-					(reference "R129")
-					(unit 1)
-				)
-				(path "/838bf11c-36b7-41d7-9462-fe98a188d617/d7ed326e-dbc5-4110-8331-7e3bdacabdbd"
-					(reference "R131")
-					(unit 1)
-				)
-				(path "/838bf11c-36b7-41d7-9462-fe98a188d617/9caee5f1-c259-48c3-ab00-5902eb9cdfc4"
-					(reference "R136")
+					(reference "R25")
+					(unit 1)
+				)
+				(path "/838bf11c-36b7-41d7-9462-fe98a188d617/d7ed326e-dbc5-4110-8331-7e3bdacabdbd"
+					(reference "R27")
+					(unit 1)
+				)
+				(path "/838bf11c-36b7-41d7-9462-fe98a188d617/9caee5f1-c259-48c3-ab00-5902eb9cdfc4"
+					(reference "R32")
 					(unit 1)
 				)
@@
 		(on_board yes)
 		(dnp no)
-		(property "Reference" "R130"
+		(property "Reference" "R26"
 			(at 149.86 72.644 90)
 			(effects
@@
 			(project "femta-control"
 				(path "/838bf11c-36b7-41d7-9462-fe98a188d617/d7ed326e-dbc5-4110-8331-7e3bdacabdbd"
-					(reference "R130")
-					(unit 1)
-				)
-				(path "/838bf11c-36b7-41d7-9462-fe98a188d617/2005ce18-3dfb-489b-ad6c-5d04a90f0ec8"
-					(reference "R128")
-					(unit 1)
-				)
-				(path "/838bf11c-36b7-41d7-9462-fe98a188d617/9caee5f1-c259-48c3-ab00-5902eb9cdfc4"
-					(reference "R135")
+					(reference "R26")
+					(unit 1)
+				)
+				(path "/838bf11c-36b7-41d7-9462-fe98a188d617/2005ce18-3dfb-489b-ad6c-5d04a90f0ec8"
+					(reference "R24")
+					(unit 1)
+				)
+				(path "/838bf11c-36b7-41d7-9462-fe98a188d617/9caee5f1-c259-48c3-ab00-5902eb9cdfc4"
+					(reference "R31")
 					(unit 1)
 				)
@@
 		(on_board yes)
 		(dnp no)
-		(property "Reference" "#PWR0139"
+		(property "Reference" "#PWR044"
 			(at 107.95 88.9 0)
 			(effects
@@
 			(project "femta-control"
 				(path "/838bf11c-36b7-41d7-9462-fe98a188d617/d7ed326e-dbc5-4110-8331-7e3bdacabdbd"
-					(reference "#PWR0139")
-					(unit 1)
-				)
-				(path "/838bf11c-36b7-41d7-9462-fe98a188d617/2005ce18-3dfb-489b-ad6c-5d04a90f0ec8"
-					(reference "#PWR0137")
-					(unit 1)
-				)
-				(path "/838bf11c-36b7-41d7-9462-fe98a188d617/9caee5f1-c259-48c3-ab00-5902eb9cdfc4"
-					(reference "#PWR0143")
+					(reference "#PWR044")
+					(unit 1)
+				)
+				(path "/838bf11c-36b7-41d7-9462-fe98a188d617/2005ce18-3dfb-489b-ad6c-5d04a90f0ec8"
+					(reference "#PWR042")
+					(unit 1)
+				)
+				(path "/838bf11c-36b7-41d7-9462-fe98a188d617/9caee5f1-c259-48c3-ab00-5902eb9cdfc4"
+					(reference "#PWR048")
 					(unit 1)
 				)
@@
 		(on_board yes)
 		(dnp no)
-		(property "Reference" "#PWR0138"
+		(property "Reference" "#PWR043"
 			(at 123.19 125.73 0)
 			(effects
@@
 			(project "femta-control"
 				(path "/838bf11c-36b7-41d7-9462-fe98a188d617/2005ce18-3dfb-489b-ad6c-5d04a90f0ec8"
-					(reference "#PWR0138")
-					(unit 1)
-				)
-				(path "/838bf11c-36b7-41d7-9462-fe98a188d617/d7ed326e-dbc5-4110-8331-7e3bdacabdbd"
-					(reference "#PWR0140")
-					(unit 1)
-				)
-				(path "/838bf11c-36b7-41d7-9462-fe98a188d617/9caee5f1-c259-48c3-ab00-5902eb9cdfc4"
-					(reference "#PWR0144")
-					(unit 1)
-				)
+					(reference "#PWR043")
+					(unit 1)
+				)
+				(path "/838bf11c-36b7-41d7-9462-fe98a188d617/d7ed326e-dbc5-4110-8331-7e3bdacabdbd"
+					(reference "#PWR045")
+					(unit 1)
+				)
+				(path "/838bf11c-36b7-41d7-9462-fe98a188d617/9caee5f1-c259-48c3-ab00-5902eb9cdfc4"
+					(reference "#PWR049")
+					(unit 1)
+				)

Commit message: schematic finished milestone
Parts:
- renumbered C19 to C20, R25 to R34, R26 to R35
Changed lines of the file:
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@@
 		(on_board yes)
 		(dnp no)
-		(property "Reference" "C19"
+		(property "Reference" "C20"
 			(at 110.49 77.47 0)
 			(effects
@@
 			(project "femta-control"
 				(path "/838bf11c-36b7-41d7-9462-fe98a188d617/d7ed326e-dbc5-4110-8331-7e3bdacabdbd"
+					(reference "C20")
+					(unit 1)
+				)
+				(path "/838bf11c-36b7-41d7-9462-fe98a188d617/2005ce18-3dfb-489b-ad6c-5d04a90f0ec8"
 					(reference "C19")
 					(unit 1)
 				)
-				(path "/838bf11c-36b7-41d7-9462-fe98a188d617/2005ce18-3dfb-489b-ad6c-5d04a90f0ec8"
-					(reference "C18")
-					(unit 1)
-				)
-				(path "/838bf11c-36b7-41d7-9462-fe98a188d617/9caee5f1-c259-48c3-ab00-5902eb9cdfc4"
-					(reference "C21")
+				(path "/838bf11c-36b7-41d7-9462-fe98a188d617/9caee5f1-c259-48c3-ab00-5902eb9cdfc4"
+					(reference "C22")
 					(unit 1)
 				)
@@
 		(on_board yes)
 		(dnp no)
-		(property "Reference" "R25"
+		(property "Reference" "R34"
 			(at 157.48 85.09 0)
 			(effects
@@
 			(project "femta-control"
 				(path "/838bf11c-36b7-41d7-9462-fe98a188d617/2005ce18-3dfb-489b-ad6c-5d04a90f0ec8"
-					(reference "R25")
-					(unit 1)
-				)
-				(path "/838bf11c-36b7-41d7-9462-fe98a188d617/d7ed326e-dbc5-4110-8331-7e3bdacabdbd"
-					(reference "R27")
-					(unit 1)
-				)
-				(path "/838bf11c-36b7-41d7-9462-fe98a188d617/9caee5f1-c259-48c3-ab00-5902eb9cdfc4"
-					(reference "R32")
+					(reference "R34")
+					(unit 1)
+				)
+				(path "/838bf11c-36b7-41d7-9462-fe98a188d617/d7ed326e-dbc5-4110-8331-7e3bdacabdbd"
+					(reference "R36")
+					(unit 1)
+				)
+				(path "/838bf11c-36b7-41d7-9462-fe98a188d617/9caee5f1-c259-48c3-ab00-5902eb9cdfc4"
+					(reference "R41")
 					(unit 1)
 				)
@@
 		(on_board yes)
 		(dnp no)
-		(property "Reference" "R26"
+		(property "Reference" "R35"
 			(at 149.86 72.644 90)
 			(effects
@@
 			(project "femta-control"
 				(path "/838bf11c-36b7-41d7-9462-fe98a188d617/d7ed326e-dbc5-4110-8331-7e3bdacabdbd"
-					(reference "R26")
-					(unit 1)
-				)
-				(path "/838bf11c-36b7-41d7-9462-fe98a188d617/2005ce18-3dfb-489b-ad6c-5d04a90f0ec8"
-					(reference "R24")
-					(unit 1)
-				)
-				(path "/838bf11c-36b7-41d7-9462-fe98a188d617/9caee5f1-c259-48c3-ab00-5902eb9cdfc4"
-					(reference "R31")
+					(reference "R35")
+					(unit 1)
+				)
+				(path "/838bf11c-36b7-41d7-9462-fe98a188d617/2005ce18-3dfb-489b-ad6c-5d04a90f0ec8"
+					(reference "R33")
+					(unit 1)
+				)
+				(path "/838bf11c-36b7-41d7-9462-fe98a188d617/9caee5f1-c259-48c3-ab00-5902eb9cdfc4"
+					(reference "R40")
 					(unit 1)
 				)
@@
 		(on_board yes)
 		(dnp no)
-		(property "Reference" "#PWR044"
+		(property "Reference" "#PWR045"
 			(at 107.95 88.9 0)
 			(effects
@@
 			(project "femta-control"
 				(path "/838bf11c-36b7-41d7-9462-fe98a188d617/d7ed326e-dbc5-4110-8331-7e3bdacabdbd"
-					(reference "#PWR044")
-					(unit 1)
-				)
-				(path "/838bf11c-36b7-41d7-9462-fe98a188d617/2005ce18-3dfb-489b-ad6c-5d04a90f0ec8"
-					(reference "#PWR042")
-					(unit 1)
-				)
-				(path "/838bf11c-36b7-41d7-9462-fe98a188d617/9caee5f1-c259-48c3-ab00-5902eb9cdfc4"
-					(reference "#PWR048")
+					(reference "#PWR045")
+					(unit 1)
+				)
+				(path "/838bf11c-36b7-41d7-9462-fe98a188d617/2005ce18-3dfb-489b-ad6c-5d04a90f0ec8"
+					(reference "#PWR043")
+					(unit 1)
+				)
+				(path "/838bf11c-36b7-41d7-9462-fe98a188d617/9caee5f1-c259-48c3-ab00-5902eb9cdfc4"
+					(reference "#PWR049")
 					(unit 1)
 				)
@@
 		(on_board yes)
 		(dnp no)
-		(property "Reference" "#PWR043"
+		(property "Reference" "#PWR044"
 			(at 123.19 125.73 0)
 			(effects
@@
 			(project "femta-control"
 				(path "/838bf11c-36b7-41d7-9462-fe98a188d617/2005ce18-3dfb-489b-ad6c-5d04a90f0ec8"
-					(reference "#PWR043")
-					(unit 1)
-				)
-				(path "/838bf11c-36b7-41d7-9462-fe98a188d617/d7ed326e-dbc5-4110-8331-7e3bdacabdbd"
-					(reference "#PWR045")
-					(unit 1)
-				)
-				(path "/838bf11c-36b7-41d7-9462-fe98a188d617/9caee5f1-c259-48c3-ab00-5902eb9cdfc4"
-					(reference "#PWR049")
-					(unit 1)
-				)
+					(reference "#PWR044")
+					(unit 1)
+				)
+				(path "/838bf11c-36b7-41d7-9462-fe98a188d617/d7ed326e-dbc5-4110-8331-7e3bdacabdbd"
+					(reference "#PWR046")
+					(unit 1)
+				)
+				(path "/838bf11c-36b7-41d7-9462-fe98a188d617/9caee5f1-c259-48c3-ab00-5902eb9cdfc4"
+					(reference "#PWR050")
+					(unit 1)
+				)

Commit message: capacitor footprints
Parts:
- C20: footprint (none) -> Capacitor_SMD:C_0603_1608Metric
Changed lines of the file:
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@@
 			)
 		)
-		(property "Footprint" ""
+		(property "Footprint" "Capacitor_SMD:C_0603_1608Metric"
 			(at 108.9152 82.55 0)
 			(effects

Commit message: add more footprints
Parts:
- R34: footprint (none) -> Resistor_SMD:R_0603_1608Metric
Changed lines of the file:
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@@
 			)
 		)
-		(property "Footprint" ""
+		(property "Footprint" "Resistor_SMD:R_0603_1608Metric"
 			(at 154.432 85.09 90)
 			(effects

Commit message: footprint selection
Parts:
- R35: footprint (none) -> Resistor_SMD:R_0805_2012Metric
Changed lines of the file:
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@@
 			)
 		)
-		(property "Footprint" ""
+		(property "Footprint" "Resistor_SMD:R_0805_2012Metric"
 			(at 149.86 76.708 90)
 			(effects
