File: thermal-master.kicad_sch (KiCad schematic)
At the start: 29 parts, among them U48 SN74HCS595-Q1, U49 SN74HCS165-Q1, U51 SN74HCS595-Q1, U52 TPS7A91, U53 LM358-N-Q1, U54 MCP3208, U55 MCP3208, U64 LTC2620IGN, U67 SN74LVC2G125

Commit message: work
Other:
- sheet FEMTA Thermal Circuit 1 ports: added none; removed HEATER+, THERM+
- sheet FEMTA Thermal Circuit 2 ports: added none; removed HEATER+, THERM+
- sheet FEMTA Thermal Circuit 3 ports: added none; removed HEATER+, THERM+
- sheet FEMTA Thermal Circuit 4 ports: added none; removed HEATER+, THERM+
- sheet FEMTA Thermal Circuit 5 ports: added none; removed HEATER+, THERM+
- sheet FEMTA Thermal Circuit 6 ports: added none; removed HEATER+, THERM+
- sheet Tank Thermal Circuit ports: added none; removed HEATER+, THERM+

Commit message: 540 COMPONENTS I AM LOSING MY MINDDDDDD
Parts:
- renumbered C100 to C64, C101 to C65, C97 to C66, C120 to C67, C102 to C68, C103 to C69, C96 to C70, C98 to C71, C114 to C72, C115 to C73, C116 to C74, C112 to C75, C117 to C76, C113 to C77, R235 to R110, R236 to R111, R234 to R112, R257 to R113, U53 to U67, U52 to U68, U67 to U69, U49 to U70, U48 to U71, U51 to U72, U54 to U73, U55 to U74, U64 to U75
Connections:
- net +3.3V: now also R112.1
- net +5V: no longer R112.1
- net ADC1_CS renamed T_ADC_CS
- net ADC2_CS renamed P_ADC_CS
- net DAC1_CS renamed TSET_CS
- net EN_OUTPUTS renamed EN_OUT_595
- net LOAD_HTR_STATES renamed LOAD_165
- net LOAD_OUTPUTS renamed LOAD_595
Other:
- moved on the sheet: C66, C67, C70, C71, C74, C76, R112, U69, U70, U71, U72, U74

Commit message: schematic finished milestone
Parts:
- added C91, C95: 10uF, symbol Device:C
- C90: renamed from C73; value 0.1uF -> 1uF
- C94: renamed from C76; value 0.1uF -> 1uF
- renumbered C64 to C81, C65 to C82, C66 to C83, C67 to C84, C68 to C85, C69 to C86, C70 to C87, C71 to C88, C72 to C89, C74 to C92, C75 to C93, C77 to C96, R110 to R119, R111 to R120, R112 to R121, R113 to R122
Connections:
- net +3.3V: now also C91.1, C95.1
- net GND: now also C91.2, C95.2
Other:
- moved on the sheet: C90, C94

Commit message: capacitor footprints
Parts:
- C81, C85, C91, C95: footprint (none) -> Capacitor_SMD:C_0805_2012Metric
- C82, C83, C84, C86, C87, C88, C89, C90, C92, C93, C94, C96: footprint (none) -> Capacitor_SMD:C_0603_1608Metric
- U67: footprint (none) -> Package_SO:SOIC-8_3.9x4.9mm_P1.27mm
Changed lines of the file:
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@@
 			)
 		)
-		(property "Footprint" ""
+		(property "Footprint" "Capacitor_SMD:C_0603_1608Metric"
 			(at 279.0952 87.63 0)
 			(effects
@@
 			)
 		)
-		(property "Footprint" ""
+		(property "Footprint" "Capacitor_SMD:C_0603_1608Metric"
 			(at 290.5252 132.08 0)
 			(effects
@@
 			)
 		)
-		(property "Footprint" ""
+		(property "Footprint" "Capacitor_SMD:C_0603_1608Metric"
 			(at 315.9252 83.82 0)
 			(effects
@@
 			)
 		)
-		(property "Footprint" ""
+		(property "Footprint" "Capacitor_SMD:C_0603_1608Metric"
 			(at 265.1252 132.08 0)
 			(effects
@@
 			)
 		)
-		(property "Footprint" ""
+		(property "Footprint" "Capacitor_SMD:C_0603_1608Metric"
 			(at 35.2552 149.86 0)
 			(effects
@@
 			)
 		)
-		(property "Footprint" ""
+		(property "Footprint" "Capacitor_SMD:C_0603_1608Metric"
 			(at 160.9852 107.95 0)
 			(effects
@@
 			)
 		)
-		(property "Footprint" ""
+		(property "Footprint" "Capacitor_SMD:C_0805_2012Metric"
 			(at 25.0952 31.75 0)
 			(effects
@@
 			)
 		)
-		(property "Footprint" ""
+		(property "Footprint" "Capacitor_SMD:C_0603_1608Metric"
 			(at 41.6052 111.76 0)
 			(effects
@@
 			)
 		)
-		(property "Footprint" ""
+		(property "Footprint" "Package_SO:SOIC-8_3.9x4.9mm_P1.27mm"
 			(at 97.79 78.74 0)
 			(effects
@@
 			)
 		)
-		(property "Footprint" ""
+		(property "Footprint" "Package_SO:SOIC-8_3.9x4.9mm_P1.27mm"
 			(at 48.26 60.96 0)
 			(effects
@@
 			)
 		)
-		(property "Footprint" ""
+		(property "Footprint" "Capacitor_SMD:C_0603_1608Metric"
 			(at 253.6952 83.82 0)
 			(effects
@@
 			)
 		)
-		(property "Footprint" ""
+		(property "Footprint" "Capacitor_SMD:C_0603_1608Metric"
 			(at 31.4452 39.37 0)
 			(effects
@@
 			)
 		)
-		(property "Footprint" ""
+		(property "Footprint" "Capacitor_SMD:C_0805_2012Metric"
 			(at 83.5152 33.02 0)
 			(effects
@@
 			)
 		)
-		(property "Footprint" ""
+		(property "Footprint" "Package_SO:SOIC-8_3.9x4.9mm_P1.27mm"
 			(at 48.26 83.82 0)
 			(effects
@@
 			)
 		)
-		(property "Footprint" ""
+		(property "Footprint" "Capacitor_SMD:C_0603_1608Metric"
 			(at 103.8352 107.95 0)
 			(effects
@@
 			)
 		)
-		(property "Footprint" ""
+		(property "Footprint" "Capacitor_SMD:C_0805_2012Metric"
 			(at 301.9552 132.08 0)
 			(effects
@@
 			)
 		)
-		(property "Footprint" ""
+		(property "Footprint" "Capacitor_SMD:C_0603_1608Metric"
 			(at 227.0252 83.82 0)
 			(effects
@@
 			)
 		)
-		(property "Footprint" ""
+		(property "Footprint" "Capacitor_SMD:C_0603_1608Metric"
 			(at 84.7852 82.55 0)
 			(effects
@@
 			)
 		)
-		(property "Footprint" ""
+		(property "Footprint" "Capacitor_SMD:C_0805_2012Metric"
 			(at 265.1252 83.82 0)
 			(effects

Commit message: add more footprints
Parts:
- R121, R122: footprint (none) -> Resistor_SMD:R_0603_1608Metric
- RV1, RV2: footprint (none) -> femta-control:Bourns PVG3A
- U75: footprint (none) -> Package_SO:SSOP-16_3.9x4.9mm_P0.635mm
Changed lines of the file:
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@@
 			)
 		)
-		(property "Footprint" ""
+		(property "Footprint" "femta-control:Bourns PVG3A"
 			(at 31.75 81.28 0)
 			(effects
@@
 			)
 		)
-		(property "Footprint" ""
+		(property "Footprint" "Package_SO:SSOP-16_3.9x4.9mm_P0.635mm"
 			(at 302.26 87.63 0)
 			(effects
@@
 			)
 		)
-		(property "Footprint" ""
+		(property "Footprint" "femta-control:Bourns PVG3A"
 			(at 31.75 58.42 0)
 			(effects
@@
 			)
 		)
-		(property "Footprint" ""
+		(property "Footprint" "Resistor_SMD:R_0603_1608Metric"
 			(at 104.648 124.46 90)
 			(effects
@@
 			)
 		)
-		(property "Footprint" ""
+		(property "Footprint" "Resistor_SMD:R_0603_1608Metric"
 			(at 291.338 88.9 90)
 			(effects

Commit message: footprint selection
Parts:
- R119, R120: footprint (none) -> Resistor_SMD:R_0603_1608Metric
Changed lines of the file:
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@@
 			)
 		)
-		(property "Footprint" ""
+		(property "Footprint" "Resistor_SMD:R_0603_1608Metric"
 			(at 62.992 30.48 90)
 			(effects
@@
 			)
 		)
-		(property "Footprint" ""
+		(property "Footprint" "Resistor_SMD:R_0603_1608Metric"
 			(at 73.66 28.448 90)
 			(effects
